Commit message: Refactor robot simulation to two-wheel diff drive
Move Gazebo-specific physics, lidar, and DiffDrive configuration into a native SDF model while keeping the URDF/xacro focused on ROS TF and RViz visualization.

Replace the four-wheel skid-steer layout with left/right drive wheels and a passive caster to reduce lateral slip during in-place rotation and improve SLAM odometry consistency.

Spawn the Gazebo model from model.sdf, install the new model assets, and tighten package dependencies / install directories for cleaner builds.

File: src/my_robot_description/urdf/my_robot.urdf.xacro (robot description, xacro)
@@ -9,7 +9,9 @@
   <xacro:property name="wheel_radius" value="0.08"/>
   <xacro:property name="wheel_width" value="0.04"/>
-  <xacro:property name="wheel_x_offset" value="0.21"/>
   <xacro:property name="wheel_y_offset" value="0.23"/>
   <xacro:property name="wheel_z_offset" value="-0.045"/>
+  <xacro:property name="caster_x_offset" value="-0.24"/>
+  <xacro:property name="caster_radius" value="0.04"/>
+  <xacro:property name="caster_z_offset" value="-0.08"/>
   <xacro:property name="laser_radius" value="0.07"/>
   <xacro:property name="laser_height" value="0.05"/>
@@ -22,4 +24,7 @@
   <material name="black">
     <color rgba="0.02 0.02 0.02 1.0"/>
+  </material>
+  <material name="gray">
+    <color rgba="0.45 0.45 0.45 1.0"/>
   </material>
   <material name="red">
@@ -90,10 +95,36 @@
   </xacro:macro>
   <!-- ===================== -->
-  <!-- Four wheels -->
+  <!-- Two differential-drive wheels -->
   <!-- ===================== -->
-  <xacro:wheel name="left_front_wheel"  x="${wheel_x_offset}"  y="${wheel_y_offset}"/>
-  <xacro:wheel name="left_rear_wheel"   x="${-wheel_x_offset}" y="${wheel_y_offset}"/>
-  <xacro:wheel name="right_front_wheel" x="${wheel_x_offset}"  y="${-wheel_y_offset}"/>
-  <xacro:wheel name="right_rear_wheel"  x="${-wheel_x_offset}" y="${-wheel_y_offset}"/>
+  <xacro:wheel name="left_wheel"  x="0.0" y="${wheel_y_offset}"/>
+  <xacro:wheel name="right_wheel" x="0.0" y="${-wheel_y_offset}"/>
+  <!-- ===================== -->
+  <!-- Passive caster support -->
+  <!-- ===================== -->
+  <joint name="caster_joint" type="fixed">
+    <parent link="base_link"/>
+    <child link="caster_link"/>
+    <origin xyz="${caster_x_offset} 0 ${caster_z_offset}" rpy="0 0 0"/>
+  </joint>
+  <link name="caster_link">
+    <visual>
+      <geometry>
+        <sphere radius="${caster_radius}"/>
+      </geometry>
+      <material name="gray"/>
+    </visual>
+    <collision>
+      <geometry>
+        <sphere radius="${caster_radius}"/>
+      </geometry>
+    </collision>
+    <inertial>
+      <mass value="0.2"/>
+      <inertia
+        ixx="0.0002" ixy="0.0" ixz="0.0"
+        iyy="0.0002" iyz="0.0"
+        izz="0.0002"/>
+    </inertial>
+  </link>
   <!-- ===================== -->
   <!-- Laser lidar -->
@@ -124,77 +155,3 @@
     </inertial>
   </link>
-  <!-- ===================== -->
-  <!-- Gazebo diff drive -->
-  <!-- ===================== -->
-  <gazebo>
-    <plugin
-      filename="gz-sim-diff-drive-system"
-      name="gz::sim::systems::DiffDrive">
-      <left_joint>left_front_wheel_joint</left_joint>
-      <left_joint>left_rear_wheel_joint</left_joint>
-      <right_joint>right_front_wheel_joint</right_joint>
-      <right_joint>right_rear_wheel_joint</right_joint>
-      <wheel_separation>${2 * wheel_y_offset}</wheel_separation>
-      <wheel_radius>${wheel_radius}</wheel_radius>
-      <odom_publish_frequency>50</odom_publish_frequency>
-      <max_velocity>1.0</max_velocity>
-      <max_acceleration>0.8</max_acceleration>
-      <max_jerk>2.0</max_jerk>
-      <topic>/cmd_vel</topic>
-      <odom_topic>/odom</odom_topic>
-      <frame_id>odom</frame_id>
-      <child_frame_id>base_footprint</child_frame_id>
-    </plugin>
-  </gazebo>
-  <!-- Keep wheel contact predictable in simulation. Low side friction helps a
-       skid-steer/four-wheel diff robot turn without dragging odometry away. -->
-  <gazebo reference="left_front_wheel_link">
-    <mu1>1.0</mu1>
-    <mu2>0.2</mu2>
-  </gazebo>
-  <gazebo reference="left_rear_wheel_link">
-    <mu1>1.0</mu1>
-    <mu2>0.2</mu2>
-  </gazebo>
-  <gazebo reference="right_front_wheel_link">
-    <mu1>1.0</mu1>
-    <mu2>0.2</mu2>
-  </gazebo>
-  <gazebo reference="right_rear_wheel_link">
-    <mu1>1.0</mu1>
-    <mu2>0.2</mu2>
-  </gazebo>
-  <!-- ===================== -->
-  <!-- Gazebo lidar sensor -->
-  <!-- ===================== -->
-  <gazebo reference="base_link">
-    <sensor name="laser_sensor" type="gpu_lidar">
-      <pose>0.20 0 0.13 0 0 0</pose>
-      <topic>/scan</topic>
-      <update_rate>10</update_rate>
-      <gz_frame_id>laser_link</gz_frame_id>
-      <ray>
-        <scan>
-          <horizontal>
-            <samples>360</samples>
-            <resolution>1</resolution>
-            <min_angle>-3.14159</min_angle>
-            <max_angle>3.14159</max_angle>
-          </horizontal>
-        </scan>
-        <range>
-          <min>0.12</min>
-          <max>10.0</max>
-          <resolution>0.01</resolution>
-        </range>
-        <noise>
-          <type>gaussian</type>
-          <mean>0.0</mean>
-          <stddev>0.01</stddev>
-        </noise>
-      </ray>
-      <always_on>true</always_on>
-      <visualize>true</visualize>
-    </sensor>
-  </gazebo>
 </robot>

Commit message: Tune robot geometry and wheel direction
Align the two-wheel differential-drive model dimensions so the drive wheels sit on the ground and the lidar rests on the base top instead of floating.

Reverse the wheel joint axes so positive DiffDrive wheel velocity should move the robot toward its +x / lidar-facing direction.

Reduce DiffDrive acceleration and jerk limits to make stop commands less likely to destabilize Gazebo contact physics.

File: src/my_robot_description/urdf/my_robot.urdf.xacro (robot description, xacro)
@@ -10,5 +10,5 @@
   <xacro:property name="wheel_width" value="0.04"/>
   <xacro:property name="wheel_y_offset" value="0.23"/>
-  <xacro:property name="wheel_z_offset" value="-0.045"/>
+  <xacro:property name="wheel_z_offset" value="-0.04"/>
   <xacro:property name="caster_x_offset" value="-0.24"/>
   <xacro:property name="caster_radius" value="0.04"/>
@@ -71,5 +71,5 @@
       <child link="${name}_link"/>
       <origin xyz="${x} ${y} ${wheel_z_offset}" rpy="${pi/2} 0 0"/>
-      <axis xyz="0 0 1"/>
+      <axis xyz="0 0 -1"/>
     </joint>
     <link name="${name}_link">
@@ -133,5 +133,5 @@
     <parent link="base_link"/>
     <child link="laser_link"/>
-    <origin xyz="0.20 0 0.13" rpy="0 0 0"/>
+    <origin xyz="0.20 0 0.10" rpy="0 0 0"/>
   </joint>
   <link name="laser_link">

Commit message: Stabilize caster and teleop stopping
Replace the fixed sphere caster with a passive swivel-and-wheel caster in both the ROS visualization model and Gazebo SDF model.

Tune caster friction and joint damping to reduce contact impulses during braking.

Ramp keyboard stop commands down over a short interval instead of publishing an abrupt zero velocity.

File: src/my_robot_description/urdf/my_robot.urdf.xacro (robot description, xacro)
@@ -13,4 +13,5 @@
   <xacro:property name="caster_x_offset" value="-0.24"/>
   <xacro:property name="caster_radius" value="0.04"/>
+  <xacro:property name="caster_width" value="0.025"/>
   <xacro:property name="caster_z_offset" value="-0.08"/>
   <xacro:property name="laser_radius" value="0.07"/>
@@ -102,13 +103,35 @@
   <!-- Passive caster support -->
   <!-- ===================== -->
-  <joint name="caster_joint" type="fixed">
+  <joint name="caster_swivel_joint" type="continuous">
     <parent link="base_link"/>
-    <child link="caster_link"/>
+    <child link="caster_swivel_link"/>
     <origin xyz="${caster_x_offset} 0 ${caster_z_offset}" rpy="0 0 0"/>
+    <axis xyz="0 0 1"/>
   </joint>
-  <link name="caster_link">
+  <link name="caster_swivel_link">
     <visual>
       <geometry>
-        <sphere radius="${caster_radius}"/>
+        <sphere radius="0.015"/>
+      </geometry>
+      <material name="gray"/>
+    </visual>
+    <inertial>
+      <mass value="0.05"/>
+      <inertia
+        ixx="0.00002" ixy="0.0" ixz="0.0"
+        iyy="0.00002" iyz="0.0"
+        izz="0.00002"/>
+    </inertial>
+  </link>
+  <joint name="caster_wheel_joint" type="continuous">
+    <parent link="caster_swivel_link"/>
+    <child link="caster_wheel_link"/>
+    <origin xyz="0 0 0" rpy="${pi/2} 0 0"/>
+    <axis xyz="0 0 1"/>
+  </joint>
+  <link name="caster_wheel_link">
+    <visual>
+      <geometry>
+        <cylinder radius="${caster_radius}" length="${caster_width}"/>
       </geometry>
       <material name="gray"/>
@@ -116,13 +139,13 @@
     <collision>
       <geometry>
-        <sphere radius="${caster_radius}"/>
+        <cylinder radius="${caster_radius}" length="${caster_width}"/>
       </geometry>
     </collision>
     <inertial>
-      <mass value="0.2"/>
+      <mass value="0.15"/>
       <inertia
-        ixx="0.0002" ixy="0.0" ixz="0.0"
-        iyy="0.0002" iyz="0.0"
-        izz="0.0002"/>
+        ixx="0.0001" ixy="0.0" ixz="0.0"
+        iyy="0.0001" iyz="0.0"
+        izz="0.0001"/>
     </inertial>
   </link>

Commit message: Normalize wheel joint axes
Keep wheel joint axes positive in both robot variants and flip the wheel link roll direction instead of relying on negative joint axes.

This keeps positive DiffDrive wheel commands aligned with the robot +x direction while avoiding the previous negative-axis configuration that may destabilize stop commands.

File: src/my_robot_description/urdf/my_robot.urdf.xacro (robot description, xacro)
@@ -71,6 +71,6 @@
       <parent link="base_link"/>
       <child link="${name}_link"/>
-      <origin xyz="${x} ${y} ${wheel_z_offset}" rpy="${pi/2} 0 0"/>
-      <axis xyz="0 0 -1"/>
+      <origin xyz="${x} ${y} ${wheel_z_offset}" rpy="${-pi/2} 0 0"/>
+      <axis xyz="0 0 1"/>
     </joint>
     <link name="${name}_link">

File: src/my_robot_description/urdf/my_robot_four_wheel.urdf.xacro (robot description, xacro)
@@ -50,6 +50,6 @@
       <parent link="base_link"/>
       <child link="${name}_link"/>
-      <origin xyz="${x} ${y} ${wheel_z_offset}" rpy="${pi/2} 0 0"/>
-      <axis xyz="0 0 -1"/>
+      <origin xyz="${x} ${y} ${wheel_z_offset}" rpy="${-pi/2} 0 0"/>
+      <axis xyz="0 0 1"/>
     </joint>
     <link name="${name}_link">

Commit message: Add car-like four-wheel teleop and tune caster robot
Add a four-wheel keyboard controller that converts speed and steering input into arc motion instead of in-place rotation.

Retune the two-wheel caster model geometry, support heights, and base inertia so the robot sits like a stable three-wheel platform.

File: src/my_robot_description/urdf/my_robot.urdf.xacro (robot description, xacro)
@@ -4,17 +4,18 @@
   <!-- Robot parameters -->
   <!-- ===================== -->
-  <xacro:property name="base_length" value="0.60"/>
-  <xacro:property name="base_width" value="0.40"/>
-  <xacro:property name="base_height" value="0.15"/>
+  <xacro:property name="base_length" value="0.56"/>
+  <xacro:property name="base_width" value="0.34"/>
+  <xacro:property name="base_height" value="0.11"/>
   <xacro:property name="wheel_radius" value="0.08"/>
-  <xacro:property name="wheel_width" value="0.04"/>
-  <xacro:property name="wheel_y_offset" value="0.23"/>
-  <xacro:property name="wheel_z_offset" value="-0.04"/>
-  <xacro:property name="caster_x_offset" value="-0.24"/>
-  <xacro:property name="caster_radius" value="0.04"/>
+  <xacro:property name="wheel_width" value="0.045"/>
+  <xacro:property name="drive_wheel_x_offset" value="-0.16"/>
+  <xacro:property name="wheel_y_offset" value="0.20"/>
+  <xacro:property name="wheel_z_offset" value="-0.025"/>
+  <xacro:property name="caster_x_offset" value="0.23"/>
+  <xacro:property name="caster_radius" value="0.045"/>
   <xacro:property name="caster_width" value="0.025"/>
-  <xacro:property name="caster_z_offset" value="-0.08"/>
-  <xacro:property name="laser_radius" value="0.07"/>
-  <xacro:property name="laser_height" value="0.05"/>
+  <xacro:property name="caster_z_offset" value="-0.06"/>
+  <xacro:property name="laser_radius" value="0.06"/>
+  <xacro:property name="laser_height" value="0.04"/>
   <!-- ===================== -->
   <!-- Materials -->
@@ -39,5 +40,5 @@
     <parent link="base_footprint"/>
     <child link="base_link"/>
-    <origin xyz="0 0 0.12" rpy="0 0 0"/>
+    <origin xyz="0 0 0.105" rpy="0 0 0"/>
   </joint>
   <!-- ===================== -->
@@ -59,7 +60,7 @@
       <mass value="8.0"/>
       <inertia
-        ixx="0.12" ixy="0.0" ixz="0.0"
-        iyy="0.25" iyz="0.0"
-        izz="0.30"/>
+        ixx="0.085" ixy="0.0" ixz="0.0"
+        iyy="0.217" iyz="0.0"
+        izz="0.286"/>
     </inertial>
   </link>
@@ -98,6 +99,6 @@
   <!-- Two differential-drive wheels -->
   <!-- ===================== -->
-  <xacro:wheel name="left_wheel"  x="0.0" y="${wheel_y_offset}"/>
-  <xacro:wheel name="right_wheel" x="0.0" y="${-wheel_y_offset}"/>
+  <xacro:wheel name="left_wheel"  x="${drive_wheel_x_offset}" y="${wheel_y_offset}"/>
+  <xacro:wheel name="right_wheel" x="${drive_wheel_x_offset}" y="${-wheel_y_offset}"/>
   <!-- ===================== -->
   <!-- Passive caster support -->
@@ -156,5 +157,5 @@
     <parent link="base_link"/>
     <child link="laser_link"/>
-    <origin xyz="0.20 0 0.10" rpy="0 0 0"/>
+    <origin xyz="0.14 0 0.08" rpy="0 0 0"/>
   </joint>
   <link name="laser_link">
